File: PCB/Voice assistant for HA.kicad_pcb (KiCad board)
At the start: 2 copper layers, 75.1 x 44.6 mm, 33 parts, among them J1 Conn_01x06_Pin, J2 Screw_Terminal_01x02, J3 Conn_01x03_Pin, J4 Conn_01x03_Pin, J5 Conn_01x03_Pin, J6 Conn_01x03_Pin, U1 AMS1117-3.3, U2 ESP32-S3-WROOM-1, U3 MAX98357A

Commit message: post-assembly adjustments
Parts:
- added FB2: 600R, Inductor_SMD:L_0805_2012Metric, F.Cu at (167.9, 72.5)
- moved FB1 1.08 mm to (167.9, 70.2), turned to 0 degrees
Connections:
- FB1 pad 1: Net-(J2-Pin_1) -> Net-(U3-OUTN)
- U3 pad 10: Net-(J2-Pin_2) -> Net-(U3-OUTN)
- U3 pad 9: Net-(J2-Pin_1) -> Net-(U3-OUTP)
Routing:
- net Net-(J2-Pin_2): track 20.8 -> 15.8 mm
- net Net-(J2-Pin_1): track 15.2 -> 10.9 mm
- net Net-(U3-OUTN): track 0.00 -> 3.00 mm
- net Net-(U3-OUTP): track 0.00 -> 2.64 mm
Changed lines of the file:
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@@
 			(outputformat 1)
 			(mirror no)
-			(drillshape 1)
+			(drillshape 0)
 			(scaleselection 1)
-			(outputdirectory "")
+			(outputdirectory "C:/Users/já/Documents/GitHub/Voice-assistant-for-HA/Production/Gerbers/")
 		)
 	)
@@
 	(net 51 "Net-(J1-Pin_5)")
 	(net 52 "Net-(J1-Pin_6)")
+	(net 53 "Net-(U3-OUTN)")
+	(net 54 "Net-(U3-OUTP)")
 	(footprint "footprints:SW_TS-1088-AR02016"
 		(layer "F.Cu")
@@
 	(footprint "Inductor_SMD:L_0805_2012Metric"
 		(layer "F.Cu")
-		(at 168 71.325 90)
+		(at 167.95 70.25)
 		(descr "Inductor SMD 0805 (2012 Metric), square (rectangular) end terminal, IPC-7351 nominal, (Body size source: IPC-SM-782 page 80, https://www.pcb-3d.com/wordpress/wp-content/uploads/ipc-sm-782a_amendment_1_and_2.pdf), generated with kicad-footprint-generator")
 		(tags "inductor")
 		(property "Reference" "FB1"
-			(at 0 -1.55 90)
+			(at 0 -1.55 0)
 			(layer "F.SilkS")
 			(effects
@@
 		)
 		(property "Value" "600R"
-			(at 0 1.55 90)
+			(at 0 1.55 0)
 			(layer "F.Fab")
 			(effects
@@
 		)
 		(property "Datasheet" "~"
-			(at 0 0 90)
+			(at 0 0 0)
 			(layer "F.Fab")
 			(hide yes)
@@
 		)
 		(property "Description" "Ferrite bead"
-			(at 0 0 90)
+			(at 0 0 0)
 			(layer "F.Fab")
 			(hide yes)
@@
 		)
 		(fp_text user "${REFERENCE}"
-			(at 0 0 90)
+			(at 0 0 0)
 			(layer "F.Fab")
 			(effects
@@
 		)
 		(pad "1" smd roundrect
-			(at -1.0625 0 90)
+			(at -1.0625 0)
 			(size 0.875 1.2)
 			(layers "F.Cu" "F.Mask" "F.Paste")
 			(roundrect_rratio 0.25)
-			(net 6 "Net-(J2-Pin_1)")
+			(net 53 "Net-(U3-OUTN)")
 			(pintype "passive")
 		)
 		(pad "2" smd roundrect
-			(at 1.0625 0 90)
+			(at 1.0625 0)
 			(size 0.875 1.2)
 			(layers "F.Cu" "F.Mask" "F.Paste")
@@
 		(embedded_fonts no)
 	)
+	(footprint "Inductor_SMD:L_0805_2012Metric"
+		(layer "F.Cu")
+		(at 167.95 72.525 180)
+		(descr "Inductor SMD 0805 (2012 Metric), square (rectangular) end terminal, IPC-7351 nominal, (Body size source: IPC-SM-782 page 80, https://www.pcb-3d.com/wordpress/wp-content/uploads/ipc-sm-782a_amendment_1_and_2.pdf), generated with kicad-footprint-generator")
+		(tags "inductor")
+		(property "Reference" "FB2"
+			(at 0 -1.55 0)
+			(layer "F.SilkS")
+			(effects
+				(font
+					(size 1 1)
+					(thickness 0.15)
+				)
+			)
+		)
+		(property "Value" "600R"
+			(at 0 1.55 0)
+			(layer "F.Fab")
+			(effects
+				(font
+					(size 1 1)
+					(thickness 0.15)
+				)
+			)
+		)
+		(property "Datasheet" "~"
+			(at 0 0 0)
+			(layer "F.Fab")
+			(hide yes)
+			(effects
+				(font
+					(size 1.27 1.27)
+					(thickness 0.15)
+				)
+			)
+		)
+		(property "Description" "Ferrite bead"
+			(at 0 0 0)
+			(layer "F.Fab")
+			(hide yes)
+			(effects
+				(font
+					(size 1.27 1.27)
+					(thickness 0.15)
+				)
+			)
+		)
+		(property ki_fp_filters "Inductor_* L_* *Ferrite*")
+		(sheetname "/")
+		(sheetfile "Voice assistant for HA.kicad_sch")
+		(attr smd)
+		(fp_line
+			(start -0.399622 0.56)
+			(end 0.399622 0.56)
+			(stroke
+				(width 0.12)
+				(type solid)
+			)
+			(layer "F.SilkS")
+		)
+		(fp_line
+			(start -0.399622 -0.56)
+			(end 0.399622 -0.56)
+			(stroke
+				(width 0.12)
+				(type solid)
+			)
+			(layer "F.SilkS")
+		)
+		(fp_rect
+			(start -1.75 -0.85)
+			(end 1.75 0.85)
+			(stroke
+				(width 0.05)
+				(type solid)
+			)
+			(fill no)
+			(layer "F.CrtYd")
+		)
+		(fp_rect
+			(start -1 -0.45)
+			(end 1 0.45)
+			(stroke
+				(width 0.1)
+				(type solid)
+			)
+			(fill no)
+			(layer "F.Fab")
+		)
+		(fp_text user "${REFERENCE}"
+			(at 0 0 0)
+			(layer "F.Fab")
+			(effects
+				(font
+					(size 0.5 0.5)
+					(thickness 0.08)
+				)
+			)
+		)
+		(pad "1" smd roundrect
+			(at -1.0625 0 180)
+			(size 0.875 1.2)
+			(layers "F.Cu" "F.Mask" "F.Paste")
+			(roundrect_rratio 0.25)
+			(net 6 "Net-(J2-Pin_1)")
+			(pintype "passive")
+		)
+		(pad "2" smd roundrect
+			(at 1.0625 0 180)
+			(size 0.875 1.2)
+			(layers "F.Cu" "F.Mask" "F.Paste")
+			(roundrect_rratio 0.25)
+			(net 54 "Net-(U3-OUTP)")
+			(pintype "passive")
+		)
+		(embedded_fonts no)
+		(model "${KICAD9_3DMODEL_DIR}/Inductor_SMD.3dshapes/L_0805_2012Metric.step"
+			(offset
+				(xyz 0 0 0)
+			)
+			(scale
+				(xyz 1 1 1)
+			)
+			(rotate
+				(xyz 0 0 0)
+			)
+		)
+	)
 	(footprint "Capacitor_Tantalum_SMD:CP_EIA-3216-18_Kemet-A"
 		(layer "F.Cu")
@@
 			(layers "F.Cu" "F.Mask" "F.Paste")
 			(roundrect_rratio 0.25)
-			(net 6 "Net-(J2-Pin_1)")
+			(net 54 "Net-(U3-OUTP)")
 			(pinfunction "OUTP")
 			(pintype "output")
@@
 			(layers "F.Cu" "F.Mask" "F.Paste")
 			(roundrect_rratio 0.25)
-			(net 5 "Net-(J2-Pin_2)")
+			(net 53 "Net-(U3-OUTN)")
 			(pinfunction "OUTN")
 			(pintype "output")
@@
 	)
 	(segment
-		(start 168 70.2625)
-		(end 171.8875 70.2625)
-		(width 0.5)
-		(layer "F.Cu")
-		(net 5)
-	)
-	(segment
 		(start 172 70.15)
 		(end 172.499938 69.650062)
@@
 	)
 	(segment
-		(start 164.4375 71.575)
-		(end 165 71.575)
-		(width 0.25)
-		(layer "F.Cu")
-		(net 5)
-	)
-	(segment
-		(start 165 71.575)
-		(end 166.3125 70.2625)
-		(width 0.25)
-		(layer "F.Cu")
-		(net 5)
-	)
-	(segment
 		(start 181.802562 69.650062)
 		(end 183.675 71.5225)
@@
 	)
 	(segment
-		(start 166.3125 70.2625)
-		(end 168 70.2625)
-		(width 0.25)
+		(start 172.499938 69.650062)
+		(end 181.802562 69.650062)
+		(width 0.5)
 		(layer "F.Cu")
 		(net 5)
 	)
 	(segment
-		(start 172.499938 69.650062)
-		(end 181.802562 69.650062)
+		(start 172 70.15)
+		(end 169.1125 70.15)
 		(width 0.5)
 		(layer "F.Cu")
@@
 	)
 	(segment
-		(start 172 72.55)
-		(end 168.1625 72.55)
+		(start 169.1125 70.15)
+		(end 169.0125 70.25)
+		(width 0.5)
+		(layer "F.Cu")
+		(net 5)
+	)
+	(segment
+		(start 169.0375 72.55)
+		(end 169.0125 72.525)
 		(width 0.5)
 		(layer "F.Cu")
@@
 	)
 	(segment
-		(start 168.1625 72.55)
-		(end 168 72.3875)
-		(width 0.5)
-		(layer "F.Cu")
-		(net 6)
-	)
-	(segment
 		(start 173.0275 71.5225)
 		(end 172 72.55)
@@
 	)
 	(segment
-		(start 164.4375 72.075)
-		(end 167.6875 72.075)
-		(width 0.25)
+		(start 172 72.55)
+		(end 169.0375 72.55)
+		(width 0.5)
 		(layer "F.Cu")
 		(net 6)
@@
 		(net 52)
 	)
+	(segment
+		(start 164.4375 71.575)
+		(end 165.5625 71.575)
+		(width 0.25)
+		(layer "F.Cu")
+		(net 53)
+	)
+	(segment
+		(start 165.5625 71.575)
+		(end 166.8875 70.25)
+		(width 0.25)
+		(layer "F.Cu")
+		(net 53)
+	)
+	(segment
+		(start 164.4375 72.075)
+		(end 166.4375 72.075)
+		(width 0.25)
+		(layer "F.Cu")
+		(net 54)
+	)
+	(segment
+		(start 166.4375 72.075)
+		(end 166.8875 72.525)
+		(width 0.25)
+		(layer "F.Cu")
+		(net 54)
+	)
 	(zone
